Commit message: made heavier so it doesnt topple so quickly

File: objects/green_box_tuned.urdf (robot description, URDF)
Before this commit: robot green_box_model, 1 links, 0 joints
Links:
- link green_box: mass 1.0 -> 10

Commit message: normal calculation with lots of debugging code, alternating arms

File: objects/green_box_tuned.urdf (robot description, URDF)
Before this commit: robot green_box_model, 1 links, 0 joints
Links:
- link green_box: geometry collision box size=0.08 0.08 0.2; visual box size=0.08 0.08 0.2

Commit message: adjusted object parameters

File: objects/green_box_tuned.urdf (robot description, URDF)
Before this commit: robot green_box_model, 1 links, 0 joints
Links:
- link green_box: mass 10 -> 2

File: objects/small_box_tuned.urdf (robot description, URDF)
Before this commit: robot small_box_model, 1 links, 0 joints
Links:
- link small_box: mass 10 -> 2

File: objects/small_box_tuned_smaller.urdf (robot description, URDF)
Before this commit: robot small_box_model, 1 links, 0 joints
Links:
- link small_box: mass 10 -> 2
