Commit message: trying heuristic approach when move_arm fails like usual

File: objects/small_box_tuned.urdf (robot description, URDF)
Before this commit: robot small_box_model, 1 links, 0 joints
Links:
- link small_box: geometry collision box size=0.07 0.07 0.14; visual box size=0.07 0.07 0.14

File: objects/small_box_tuned_smaller.urdf (robot description, URDF)
Before this commit: robot small_box_model, 1 links, 0 joints
Links:
- link small_box: geometry collision box size=0.065 0.065 0.11; visual box size=0.065 0.065 0.11
